File: Schalter-Karte_HW/Schalter-Karte_HW/source_2026-03-20/Schalter-Karte_HW.kicad_sch (KiCad schematic)
At the start: 5 parts, among them J1 MKDS 3-2 5.08, J2 MKDS 3-2 5.08, J3 MKDS 3-3 5.08, SW1 L101011MS02Q

Commit message: wip
Parts:
- removed F1: Fuse Socket, _PS_LIB_CON:Fuse Holder Littelfuse ATOF 287, symbol Device:Fuse
- removed J1, J2: MKDS 3-2 5.08, _PS_LIB_CON:MKDS_3_2_508, symbol Connector:Conn_01x02_Socket
- removed J3: MKDS 3-3 5.08, _PS_LIB_CON:MKDS_3_3_508, symbol Connector:Conn_01x03_Socket
- removed SW1: L101011MS02Q, _PS_LIB_MECH:L10101_Schiebeschalter, symbol Switch:SW_Slide_DPDT
- added F1: 3557-2, _PS_LIB_CON:Fuse Holder Littelfuse ATOF 287, symbol _PS_LIB:Fuseholder ATOF 287
- added J1: MKDS_3-2_5.08, _PS_LIB_CON:MKDS_3_2_508, symbol _PS_LIB:MKDS_3-2_5.08
- added J2: MKDS_3-3_5.08, _PS_LIB_CON:MKDS_3_3_508, symbol _PS_LIB:MKDS_3-3_5.08
- added SW1: L101011MS02Q, _PS_LIB_MECH:L10101_Schiebeschalter, symbol _PS_LIB:SW_Slide_DPDT_L101011MS02Q
Connections:
- net +24V: now also F1.1, J1.2 (Pin_2)
- net +24V_sicher: now also F1.2, SW1.2 (B), SW1.5 (B)
- net GND: now also J1.1 (Pin_1), J2.2 (Pin_2)
- new net: J2.1 (Pin_1), SW1.1 (A), SW1.6 (C)
- new net: J2.3 (Pin_3), SW1.3 (C), SW1.4 (A)

Commit message: wip
Parts:
- F1: symbol _PS_LIB:Fuseholder ATOF 287 -> Symbols:Fuseholder ATOF 287
- J1: symbol _PS_LIB:MKDS_3-2_5.08 -> Symbols:MKDS_3-2_5.08
- J2: symbol _PS_LIB:MKDS_3-3_5.08 -> Symbols:MKDS_3-3_5.08
- SW1: symbol _PS_LIB:SW_Slide_DPDT_L101011MS02Q -> Symbols:SW_Slide_DPDT_L101011MS02Q
Other:
- company: (none) -> hand-crafted-electronics
- title: (none) -> Schalter-Karte
Changed lines of the file:
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@@
 	(generator_version "9.0")
 	(paper "A4")
+	(title_block
+		(title "Schalter-Karte")
+		(date "2026-03-20")
+		(rev "V1.0")
+		(company "hand-crafted-electronics")
+		(comment 1 "https://ohwr.org/cern_ohl_s_v2.txt ")
+		(comment 2 "https://github.com/pellematrose/Schalter-Karte")
+		(comment 3 "Licensed under CERN-OHL-S v2")
+		(comment 4 "© 2026 Per-Simon Saal")
+	)
 	(junction
 		(at 130.81 88.9)
@@
 	)
 	(symbol
-		(lib_id "power:+24V")
+		(lib_id "Symbols:+24V")
 		(at 127 67.31 270)
 		(mirror x)
@@
 	)
 	(symbol
-		(lib_id "_PS_LIB:Fuseholder ATOF 287")
+		(lib_id "Symbols:Fuseholder ATOF 287")
 		(at 123.19 67.31 90)
 		(unit 1)
@@
 	)
 	(symbol
-		(lib_id "_PS_LIB:MKDS_3-3_5.08")
+		(lib_id "Symbols:MKDS_3-3_5.08")
 		(at 100.33 91.44 0)
 		(mirror y)
@@
 	)
 	(symbol
-		(lib_id "power:GND")
+		(lib_id "Symbols:GND")
 		(at 105.41 69.85 0)
 		(mirror y)
@@
 	)
 	(symbol
-		(lib_id "power:GND")
+		(lib_id "Symbols:GND")
 		(at 105.41 91.44 90)
 		(mirror x)
@@
 	)
 	(symbol
-		(lib_id "_PS_LIB:SW_Slide_DPDT_L101011MS02Q")
+		(lib_id "Symbols:SW_Slide_DPDT_L101011MS02Q")
 		(at 139.7 93.98 0)
 		(unit 1)
@@
 	)
 	(symbol
-		(lib_id "power:+24V")
+		(lib_id "Symbols:+24V")
 		(at 156.21 93.98 270)
 		(unit 1)
@@
 	)
 	(symbol
-		(lib_id "power:+24V")
+		(lib_id "Symbols:+24V")
 		(at 111.76 67.31 0)
 		(mirror y)
@@
 	)
 	(symbol
-		(lib_id "_PS_LIB:MKDS_3-2_5.08")
+		(lib_id "Symbols:MKDS_3-2_5.08")
 		(at 100.33 69.85 180)
 		(unit 1)
@@
 	)
 	(symbol
-		(lib_id "power:+24V")
+		(lib_id "Symbols:+24V")
 		(at 134.62 93.98 90)
 		(unit 1)
