File: Schalter-Karte_HW/Schalter-Karte_HW/source_2026-03-20/Schalter-Karte_HW.kicad_pcb (KiCad board)
At the start: 2 copper layers, 17.5 x 80.5 mm, 4 parts, among them J1 MKDS 3-2 5.08, J3 MKDS 3-3 5.08, SW1 L101011MS02Q

Commit message: wip
Parts:
- F1: value Fuse Socket -> 3557-2
- J1: value MKDS 3-2 5.08 -> MKDS_3-2_5.08
- J2: renamed from J3; value MKDS 3-3 5.08 -> MKDS_3-3_5.08
Connections:
- F1 pad 1: +24V_sicher -> +24V
- F1 pad 2: +24V -> +24V_sicher
Changed lines of the file:
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@@
 	(net 2 "+24V")
 	(net 3 "GND")
-	(net 4 "Net-(J3-Pin_3)")
-	(net 5 "Net-(J3-Pin_1)")
+	(net 4 "Net-(J2-Pin_3)")
+	(net 5 "Net-(J2-Pin_1)")
 	(footprint "_PS_LIB_MECH:L10101_Schiebeschalter"
 		(layer "F.Cu")
@@
 			)
 		)
+		(property "Digikey" "CKC5106-ND"
+			(at 0 0 90)
+			(unlocked yes)
+			(layer "F.Fab")
+			(hide yes)
+			(effects
+				(font
+					(size 1 1)
+					(thickness 0.15)
+				)
+			)
+		)
 		(sheetname "/")
 		(sheetfile "Schalter-Karte_HW.kicad_sch")
@@
 			(layers "*.Cu" "*.Mask")
 			(remove_unused_layers no)
-			(net 5 "Net-(J3-Pin_1)")
+			(net 5 "Net-(J2-Pin_1)")
 			(pinfunction "A")
 			(pintype "passive")
@@
 			(layers "*.Cu" "*.Mask")
 			(remove_unused_layers no)
-			(net 4 "Net-(J3-Pin_3)")
+			(net 4 "Net-(J2-Pin_3)")
 			(pinfunction "C")
 			(pintype "passive")
@@
 			(layers "*.Cu" "*.Mask")
 			(remove_unused_layers no)
-			(net 4 "Net-(J3-Pin_3)")
+			(net 4 "Net-(J2-Pin_3)")
 			(pinfunction "A")
 			(pintype "passive")
@@
 			(layers "*.Cu" "*.Mask")
 			(remove_unused_layers no)
-			(net 5 "Net-(J3-Pin_1)")
+			(net 5 "Net-(J2-Pin_1)")
 			(pinfunction "C")
 			(pintype "passive")
@@
 			)
 		)
-		(property "Value" "Fuse Socket"
+		(property "Value" "3557-2"
 			(at 0 0.25 90)
 			(layer "F.Fab")
@@
 			)
 		)
-		(property "Datasheet" "~"
+		(property "Datasheet" "https://www.keyelco.com/userAssets/file/K75p47.pdf"
 			(at 0 0 90)
 			(layer "F.Fab")
@@
 			(layers "*.Cu" "*.Mask")
 			(remove_unused_layers no)
-			(net 1 "+24V_sicher")
+			(net 2 "+24V")
 			(pintype "passive")
 			(solder_mask_margin 0.102)
@@
 			(layers "*.Cu" "*.Mask")
 			(remove_unused_layers no)
-			(net 1 "+24V_sicher")
+			(net 2 "+24V")
 			(pintype "passive")
 			(solder_mask_margin 0.102)
@@
 			(layers "*.Cu" "*.Mask")
 			(remove_unused_layers no)
-			(net 2 "+24V")
+			(net 1 "+24V_sicher")
 			(pintype "passive")
 			(solder_mask_margin 0.102)
@@
 			(layers "*.Cu" "*.Mask")
 			(remove_unused_layers no)
-			(net 2 "+24V")
+			(net 1 "+24V_sicher")
 			(pintype "passive")
 			(solder_mask_margin 0.102)
@@
 			)
 		)
-		(property "Value" "MKDS 3-2 5.08"
+		(property "Value" "MKDS_3-2_5.08"
 			(at -0.25 -6.5 0)
 			(unlocked yes)
@@
 			)
 		)
-		(property "Datasheet" "~"
+		(property "Datasheet" "https://product-download.phoenixcontact.com/2848324?response-content-disposition=inline;%20filename%3D%221711725_04_de_00.pdf%22&Expires=1774048874&Signature=iFyT5B3-womW6lKjp5XGzWeua--BUis2SV37lsN3fOwrxLgEMLrA23TCmt7nlwi7ykr87Ps5xEHVs57OHbg5HRkkk59gv3io6WeBmuQRAZV6weoNLPtYcPQeNLn5aF1XU7IeUHNLEPTX941vJscEzGtP~Ohp3b7MZL1cCDfW5h5gjoo-aowUyONotC1zxuNCCh7kpnCXrhsvQVzKOYEZP~kIA8L3KVBHTrZZ6dlP381ao0AsK~O514~kd4FiCUoDK9G-yYP6HXF56mm67ftfuCnE63yGKMlMc9a1CFPGwdcLvfi1mXo0DWzryEcO6ogvtp8cLC18eKrYcvQZf0Ukdg__&Key-Pair-Id=K1I2N54A7B0GD"
 			(at 0 0 0)
 			(layer "F.Fab")
@@
 			)
 		)
-		(property "Description" "Generic connector, single row, 01x02, script generated"
+		(property "Description" "Leiterplattenklemme, Wellenlötung, Schrauban- schluss mit Zughülse"
 			(at 0 0 0)
 			(layer "F.Fab")
@@
 			)
 		)
+		(property "Digikey" "277-1027-ND"
+			(at 0 0 180)
+			(unlocked yes)
+			(layer "F.Fab")
+			(hide yes)
+			(effects
+				(font
+					(size 1 1)
+					(thickness 0.15)
+				)
+			)
+		)
+		(property "LCSC" ""
+			(at 0 0 180)
+			(unlocked yes)
+			(layer "F.Fab")
+			(hide yes)
+			(effects
+				(font
+					(size 1 1)
+					(thickness 0.15)
+				)
+			)
+		)
+		(property "Mouser" ""
+			(at 0 0 180)
+			(unlocked yes)
+			(layer "F.Fab")
+			(hide yes)
+			(effects
+				(font
+					(size 1 1)
+					(thickness 0.15)
+				)
+			)
+		)
 		(property ki_fp_filters "Connector*:*_1x??_*")
 		(sheetname "/")
@@
 		(layer "F.Cu")
 		(at 78.25 128)
-		(property "Reference" "J3"
+		(property "Reference" "J2"
 			(at -6.75 -6.5 0)
 			(unlocked yes)
@@
 			)
 		)
-		(property "Value" "MKDS 3-3 5.08"
+		(property "Value" "MKDS_3-3_5.08"
 			(at 0 4 0)
 			(unlocked yes)
@@
 			)
 		)
-		(property "Datasheet" "~"
+		(property "Datasheet" "https://www.phoenixcontact.com/en-us/products/printed-circuit-board-terminal-mkds-3-3-508-1711738?type=pdf"
 			(at 0 0 0)
 			(layer "F.Fab")
@@
 			)
 		)
-		(property "Description" "Generic connector, single row, 01x03, script generated"
+		(property "Description" "Leiterplattenklemme, Wellenlötung, Schrauban- schluss mit Zughülse"
 			(at 0 0 0)
 			(layer "F.Fab")
@@
 			)
 		)
+		(property "Digikey" "277-1028-ND"
+			(at 0 0 0)
+			(unlocked yes)
+			(layer "F.Fab")
+			(hide yes)
+			(effects
+				(font
+					(size 1 1)
+					(thickness 0.15)
+				)
+			)
+		)
 		(property ki_fp_filters "Connector*:*_1x??_*")
 		(sheetname "/")
@@
 			(layers "*.Cu" "*.Mask")
 			(remove_unused_layers no)
-			(net 5 "Net-(J3-Pin_1)")
+			(net 5 "Net-(J2-Pin_1)")
 			(pinfunction "Pin_1")
 			(pintype "passive")
@@
 			(layers "*.Cu" "*.Mask")
 			(remove_unused_layers no)
-			(net 4 "Net-(J3-Pin_3)")
+			(net 4 "Net-(J2-Pin_3)")
 			(pinfunction "Pin_3")
 			(pintype "passive")

Commit message: wip
Parts:
- F1: footprint _PS_LIB_CON:Fuse Holder Littelfuse ATOF 287 -> Footprints:Fuse Holder Littelfuse ATOF 287
- J1: footprint _PS_LIB_CON:MKDS_3_2_508 -> Footprints:MKDS_3_2_508
- J2: footprint _PS_LIB_CON:MKDS_3_3_508 -> Footprints:MKDS_3_3_508
- SW1: footprint _PS_LIB_MECH:L10101_Schiebeschalter -> Footprints:L10101_Schiebeschalter
Changed lines of the file:
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@@
 	(net 4 "Net-(J2-Pin_3)")
 	(net 5 "Net-(J2-Pin_1)")
-	(footprint "_PS_LIB_MECH:L10101_Schiebeschalter"
+	(footprint "Footprints:L10101_Schiebeschalter"
 		(layer "F.Cu")
 		(at 78.25 110.9 90)
@@
 			)
 		)
-		(model "kicad-embed://L101011MS02Q_schiebeschalter.stp"
+		(model "${KIPRJMOD}/3dmodels/L101011MS02Q_schiebeschalter.stp"
 			(offset
 				(xyz 0 0 1.5)
@@
 		)
 	)
-	(footprint "_PS_LIB_CON:Fuse Holder Littelfuse ATOF 287"
+	(footprint "Footprints:Fuse Holder Littelfuse ATOF 287"
 		(layer "F.Cu")
 		(at 78.25 89 90)
@@
 			)
 		)
-		(model "kicad-embed://3557-2.step"
+		(model "${KIPRJMOD}/3dmodels/3557-2.step"
 			(offset
 				(xyz 0 0 0)
@@
 		)
 	)
-	(footprint "_PS_LIB_CON:MKDS_3_2_508"
+	(footprint "Footprints:MKDS_3_2_508"
 		(layer "F.Cu")
 		(at 78.25 71.5 180)
@@
 			)
 		)
-		(model "kicad-embed://1711725_06_00_MKDS-3-2-5-08_3D.stp"
+		(model "${KIPRJMOD}/3dmodels/1711725_06_00_MKDS-3-2-5-08_3D.stp"
 			(offset
 				(xyz -5.1 -5.3 0)
@@
 		)
 	)
-	(footprint "_PS_LIB_CON:MKDS_3_3_508"
+	(footprint "Footprints:MKDS_3_3_508"
 		(layer "F.Cu")
 		(at 78.25 128)
@@
 			)
 		)
-		(model "kicad-embed://1711738_06_01_MKDS-3-3-5-08_3D.stp"
+		(model "${KIPRJMOD}/3dmodels/1711738_06_01_MKDS-3-3-5-08_3D.stp"
 			(offset
 				(xyz -7.65 -5.3 0)

Commit message: wip
Parts:
- turned F1 to -90 degrees
Routing:
- net GND: track 0.00 -> 60.6 mm
- net Net-(J2-Pin_1): track 0.00 -> 28.7 mm
- net +24V_sicher: track 0.00 -> 25.1 mm
- net Net-(J2-Pin_3): track 0.00 -> 19.1 mm
- net +24V: track 0.00 -> 14.5 mm
Changed lines of the file:
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@@
 	(footprint "Footprints:Fuse Holder Littelfuse ATOF 287"
 		(layer "F.Cu")
-		(at 78.25 89 90)
+		(at 78.25 89 -90)
 		(descr "KFZ Sicherungshalter")
 		(property "Reference" "F1"
-			(at 9.5 -4.445 180)
+			(at 9.5 -4.445 0)
 			(layer "F.SilkS")
 			(effects
@@
 		(attr through_hole)
 		(fp_line
-			(start 9.905 -3.365)
-			(end -9.905 -3.365)
+			(start -9.905 3.365)
+			(end 9.905 3.365)
 			(stroke
 				(width 0.127)
@@
 		)
 		(fp_line
-			(start -9.905 -3.365)
-			(end -9.905 3.365)
+			(start 9.905 3.365)
+			(end 9.905 -3.365)
 			(stroke
 				(width 0.127)
@@
 		)
 		(fp_line
-			(start 9.905 3.365)
-			(end 9.905 -3.365)
+			(start -9.905 -3.365)
+			(end -9.905 3.365)
 			(stroke
 				(width 0.127)
@@
 		)
 		(fp_line
-			(start -9.905 3.365)
-			(end 9.905 3.365)
+			(start 9.905 -3.365)
+			(end -9.905 -3.365)
 			(stroke
 				(width 0.127)
@@
 		)
 		(fp_line
-			(start 10.155 -3.615)
-			(end 10.155 3.615)
+			(start -10.155 3.615)
+			(end -10.155 -3.615)
 			(stroke
 				(width 0.05)
@@
 		)
 		(fp_line
-			(start -10.155 -3.615)
-			(end 10.155 -3.615)
+			(start 10.155 3.615)
+			(end -10.155 3.615)
 			(stroke
 				(width 0.05)
@@
 		)
 		(fp_line
-			(start 10.155 3.615)
-			(end -10.155 3.615)
+			(start -10.155 -3.615)
+			(end 10.155 -3.615)
 			(stroke
 				(width 0.05)
@@
 		)
 		(fp_line
-			(start -10.155 3.615)
-			(end -10.155 -3.615)
+			(start 10.155 -3.615)
+			(end 10.155 3.615)
 			(stroke
 				(width 0.05)
@@
 		)
 		(fp_line
-			(start 9.905 -3.365)
-			(end -9.905 -3.365)
+			(start -9.905 3.365)
+			(end 9.905 3.365)
 			(stroke
 				(width 0.127)
@@
 		)
 		(fp_line
-			(start -9.905 -3.365)
-			(end -9.905 3.365)
+			(start 9.905 3.365)
+			(end 9.905 -3.365)
 			(stroke
 				(width 0.127)
@@
 		)
 		(fp_line
-			(start 9.905 3.365)
-			(end 9.905 -3.365)
+			(start -9.905 -3.365)
+			(end -9.905 3.365)
 			(stroke
 				(width 0.127)
@@
 		)
 		(fp_line
-			(start -9.905 3.365)
-			(end 9.905 3.365)
+			(start 9.905 -3.365)
+			(end -9.905 -3.365)
 			(stroke
 				(width 0.127)
@@
 		)
 		(pad "1" thru_hole circle
-			(at -6.735 -1.7 90)
+			(at -6.735 -1.7 270)
 			(size 2.4 2.4)
 			(drill 1.6)
@@
 		)
 		(pad "1" thru_hole circle
-			(at -6.735 1.7 90)
+			(at -6.735 1.7 270)
 			(size 2.4 2.4)
 			(drill 1.6)
@@
 		)
 		(pad "2" thru_hole circle
-			(at 6.735 -1.7 90)
+			(at 6.735 -1.7 270)
 			(size 2.4 2.4)
 			(drill 1.6)
@@
 		)
 		(pad "2" thru_hole circle
-			(at 6.735 1.7 90)
+			(at 6.735 1.7 270)
 			(size 2.4 2.4)
 			(drill 1.6)
@@
 		)
 	)
+	(segment
+		(start 78 110.9)
+		(end 81.11 110.9)
+		(width 2)
+		(layer "F.Cu")
+		(net 1)
+	)
+	(segment
+		(start 76.55 95.735)
+		(end 79.95 95.735)
+		(width 2)
+		(layer "F.Cu")
+		(net 1)
+	)
+	(segment
+		(start 76.55 95.735)
+		(end 76.55 99.55)
+		(width 2)
+		(layer "F.Cu")
+		(net 1)
+	)
+	(segment
+		(start 78.252905 101.252905)
+		(end 78.252905 110.647095)
+		(width 2)
+		(layer "F.Cu")
+		(net 1)
+	)
+	(segment
+		(start 75.39 110.9)
+		(end 78 110.9)
+		(width 2)
+		(layer "F.Cu")
+		(net 1)
+	)
+	(segment
+		(start 76.55 99.55)
+		(end 78.252905 101.252905)
+		(width 2)
+		(layer "F.Cu")
+		(net 1)
+	)
+	(segment
+		(start 78.252905 110.647095)
+		(end 78 110.9)
+		(width 2)
+		(layer "F.Cu")
+		(net 1)
+	)
+	(segment
+		(start 76.55 82.265)
+		(end 79.95 82.265)
+		(width 2)
+		(layer "F.Cu")
+		(net 2)
+	)
+	(segment
+		(start 75.71 81.425)
+		(end 76.55 82.265)
+		(width 2)
+		(layer "F.Cu")
+		(net 2)
+	)
+	(segment
+		(start 75.71 71.5)
+		(end 75.71 81.425)
+		(width 2)
+		(layer "F.Cu")
+		(net 2)
+	)
+	(segment
+		(start 78.25 123.75)
+		(end 78.25 128)
+		(width 2)
+		(layer "F.Cu")
+		(net 3)
+	)
+	(segment
+		(start 84.499 117.501)
+		(end 78.25 123.75)
+		(width 2)
+		(layer "F.Cu")
+		(net 3)
+	)
+	(segment
+		(start 84.499 75.209)
+		(end 84.499 117.501)
+		(width 2)
+		(layer "F.Cu")
+		(net 3)
+	)
+	(segment
+		(start 80.79 71.5)
+		(end 84.499 75.209)
+		(width 2)
+		(layer "F.Cu")
+		(net 3)
+	)
+	(segment
+		(start 75.39 115.5)
+		(end 81.11 115.5)
+		(width 2)
+		(layer "F.Cu")
+		(net 4)
+	)
+	(segment
+		(start 83.33 117.72)
+		(end 81.11 115.5)
+		(width 2)
+		(layer "B.Cu")
+		(net 4)
+	)
+	(segment
+		(start 83.33 128)
+		(end 83.33 117.72)
+		(width 2)
+		(layer "B.Cu")
+		(net 4)
+	)
+	(segment
+		(start 72.689 109.001)
+		(end 75.39 106.3)
+		(width 2)
+		(layer "B.Cu")
+		(net 5)
+	)
+	(segment
+		(start 72.689 127.519)
+		(end 72.689 109.001)
+		(width 2)
+		(layer "B.Cu")
+		(net 5)
+	)
+	(segment
+		(start 73.17 128)
+		(end 72.689 127.519)
+		(width 2)
+		(layer "B.Cu")
+		(net 5)
+	)
+	(segment
+		(start 75.39 106.3)
+		(end 81.11 106.3)
+		(width 2)
+		(layer "B.Cu")
+		(net 5)
+	)
 	(zone
 		(net 0)
@@
 			(pads not_allowed)
 			(copperpour not_allowed)
-			(footprints not_allowed)
+			(footprints allowed)
 		)
 		(placement
