File: Schalter-Karte_HW/Schalter-Karte_HW/source_2026-03-23/Schalter-Karte_HW.kicad_pcb (KiCad board)
At the start: 2 copper layers, 17.5 x 77 mm, 6 parts, among them J1 MKDS_3-2_5.08, J2 MKDS_3-2_5.08, SW1 L101011MS02Q

Commit message: schalter typ angepasst
Parts:
- SW1: value L101011MS02Q -> L102011MS02Q
Changed lines of the file:
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@@
 			)
 		)
-		(property "Value" "L101011MS02Q"
+		(property "Value" "L102011MS02Q"
 			(at -0.1 6.75 90)
 			(unlocked yes)
@@
 			(at 0 0 90)
 			(unlocked yes)
+			(layer "F.Fab")
+			(hide yes)
+			(effects
+				(font
+					(size 1 1)
+					(thickness 0.15)
+				)
+			)
+		)
+		(property "LCSC" ""
+			(at 0 0 90)
+			(unlocked yes)
+			(layer "F.Fab")
+			(hide yes)
+			(effects
+				(font
+					(size 1 1)
+					(thickness 0.15)
+				)
+			)
+		)
+		(property "Mouser" ""
+			(at 0 0 90)
+			(unlocked yes)
