File: Schalter-Karte_HW/Schalter-Karte_HW/source_2026-03-23/Schalter-Karte_HW.kicad_sch (KiCad schematic)
At the start: 6 parts, among them J1 MKDS_3-2_5.08, J2 MKDS_3-2_5.08, SW1 L101011MS02Q

Commit message: schalter typ angepasst
Parts:
- SW1: value L101011MS02Q -> L102011MS02Q
Changed lines of the file:
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@@
 			)
 		)
-		(property "Value" "L101011MS02Q"
+		(property "Value" "L102011MS02Q"
 			(at 139.7 86.36 0)
 			(effects
@@
 			(at 139.7 93.98 0)
 			(effects
+				(font
+					(size 1.27 1.27)
+				)
+				(hide yes)
+			)
+		)
+		(property "LCSC" ""
+			(at 139.7 93.98 0)
+			(effects
+				(font
+					(size 1.27 1.27)
+				)
+				(hide yes)
+			)
+		)
+		(property "Mouser" ""
+			(at 139.7 93.98 0)
+			(effects
